Commit message: Add the gripper tool link to the urdf

File: resources/ur5/ur5_spherized.urdf (robot description, URDF)
Before this commit: robot ur5_robotiq85, 22 links, 21 joints
Links:
- added link robotiq_85_tool_link
Joints:
- added joint robotiq_85_tool_link_joint: type fixed, parent robotiq_85_base_link, child robotiq_85_tool_link, origin xyz=0 0 0.1628 rpy=0 0 0
