Commit message: added soft cost penalties to hjcd and LS

File: resources/panda/panda.urdf (robot description, URDF)
Before this commit: robot panda, 13 links, 12 joints
Links:
- link panda_hand: geometry collision mesh filename=meshes/collision/hand.obj; visual mesh filename=meshes/visual/hand.obj
- link panda_leftfinger: geometry collision mesh filename=meshes/collision/finger.obj; visual mesh filename=meshes/visual/finger.obj
- link panda_link0: geometry collision mesh filename=meshes/collision/link0.obj; visual mesh filename=meshes/collision/link0.obj
- link panda_link1: geometry collision mesh filename=meshes/collision/link1.obj; visual mesh filename=meshes/visual/link1.obj
- link panda_link2: geometry collision mesh filename=meshes/collision/link2.obj; visual mesh filename=meshes/visual/link2.obj
- link panda_link3: geometry collision mesh filename=meshes/collision/link3.obj; visual mesh filename=meshes/visual/link3.obj
- link panda_link4: geometry collision mesh filename=meshes/collision/link4.obj; visual mesh filename=meshes/visual/link4.obj
- link panda_link5: geometry collision mesh filename=meshes/collision/link5.obj; visual mesh filename=meshes/visual/link5.obj
- link panda_link6: geometry collision mesh filename=meshes/collision/link6.obj; visual mesh filename=meshes/visual/link6.obj
- link panda_link7: geometry collision mesh filename=meshes/collision/link7.obj; visual mesh filename=meshes/collision/link7.obj
- link panda_rightfinger: geometry collision mesh filename=meshes/collision/finger.obj; visual mesh filename=meshes/visual/finger.obj
Joints:
- joint panda_finger_joint2: mimic joint=panda_finger_joint1 -> (none)

File: resources/panda/panda_spherized.urdf (robot description, URDF)
Before this commit: robot panda, 13 links, 9 joints
Joints:
- added joint panda_finger_joint1: type fixed, parent panda_hand, child panda_leftfinger, origin xyz=0 0.065 0.0584 rpy=0 0 0, axis 0 1 0
- added joint panda_finger_joint2: type fixed, parent panda_hand, child panda_rightfinger, origin xyz=0 -0.065 0.0584 rpy=0 0 0, axis 0 -1 0
- added joint panda_grasptarget_hand: type fixed, parent panda_hand, child panda_grasptarget, origin xyz=0 0 0.105 rpy=0 0 0

File: resources/ur5/ur5_spherized.urdf (robot description, URDF)
Before this commit: robot ur5_robotiq85, 23 links, 22 joints
Links:
- removed link robotiq_85_tool_link
Joints:
- removed joint robotiq_85_tool_link_joint
- joint offset_joint: origin xyz=0.0 0.0 0.0 rpy=0 0 1.57 -> xyz=0.0 0.0 0.9144 rpy=0 0 1.57
