Commit message: added coarse urdfs

File: resources/panda/panda_spherized_coarse.urdf (robot description, URDF)
Before this commit: robot panda, 13 links, 12 joints
Links:
- link panda_hand: geometry collision sphere radius=0.115569107234478; visual mesh filename=meshes/visual/hand.obj
- link panda_leftfinger: geometry collision sphere radius=0.031921979039907455; visual mesh filename=meshes/visual/finger.obj
- link panda_link0: geometry collision sphere radius=0.13297568261623383; visual mesh filename=meshes/collision/link0.obj
- link panda_link1: geometry collision sphere radius=0.15569444000720978; visual mesh filename=meshes/visual/link1.obj
- link panda_link2: geometry collision sphere radius=0.15511482954025269; visual mesh filename=meshes/visual/link2.obj
- link panda_link3: geometry collision sphere radius=0.13481484353542328; visual mesh filename=meshes/visual/link3.obj
- link panda_link4: geometry collision sphere radius=0.1361713707447052; visual mesh filename=meshes/visual/link4.obj
- link panda_link5: geometry collision sphere radius=0.1874190866947174; visual mesh filename=meshes/visual/link5.obj
- link panda_link6: geometry collision sphere radius=0.10415507107973099; visual mesh filename=meshes/visual/link6.obj
- link panda_link7: geometry collision sphere radius=0.0753609910607338; visual mesh filename=meshes/collision/link7.obj
- link panda_rightfinger: geometry collision sphere radius=0.031921979039907455; visual mesh filename=meshes/visual/finger.obj
Joints:
- joint panda_finger_joint2: mimic joint=panda_finger_joint1 -> (none)
