Commit message: huge naming refactor + scripts cleaned up

File: resources/fetch/fetch.urdf (robot description, URDF)
Before this commit: robot fetch, 17 links, 16 joints
Links:
- link base_link: geometry collision mesh filename=meshes/base_link_collision_2.stl; visual mesh filename=meshes/base_link.dae
- link bellows_link: geometry visual mesh filename=meshes/bellows_link.STL
- link elbow_flex_link: geometry collision mesh filename=meshes/elbow_flex_link_collision_2.stl; visual mesh filename=meshes/elbow_flex_link.dae
- link forearm_roll_link: geometry collision mesh filename=meshes/forearm_roll_link_collision_2.stl; visual mesh filename=meshes/forearm_roll_link.dae
- link gripper_link: geometry collision mesh filename=meshes/gripper_link_2.stl; visual mesh filename=meshes/gripper_link.dae
- link head_pan_link: geometry collision sphere radius=0.2; visual mesh filename=meshes/head_pan_link.dae
- link head_tilt_link: geometry visual mesh filename=meshes/head_tilt_link.dae
- link l_gripper_finger_link: geometry collision mesh filename=meshes/l_gripper_finger_link_2.stl; visual mesh filename=meshes/l_gripper_finger_link.STL
- link r_gripper_finger_link: geometry collision mesh filename=meshes/r_gripper_finger_link_2.stl; visual mesh filename=meshes/r_gripper_finger_link.STL
- link shoulder_lift_link: geometry collision mesh filename=meshes/shoulder_lift_link_collision_2.stl; visual mesh filename=meshes/shoulder_lift_link.dae
- link shoulder_pan_link: geometry collision mesh filename=meshes/shoulder_pan_link_collision_2.stl; visual mesh filename=meshes/shoulder_pan_link.dae
- link torso_fixed_link: geometry collision mesh filename=meshes/torso_fixed_link.STL; visual mesh filename=meshes/torso_fixed_link.dae
- link torso_lift_link: geometry collision mesh filename=meshes/torso_lift_link_split_1.stl; visual mesh filename=meshes/torso_lift_link.dae
- link upperarm_roll_link: geometry collision mesh filename=meshes/upperarm_roll_link_collision_2.stl; visual mesh filename=meshes/upperarm_roll_link.dae
- link wrist_flex_link: geometry collision mesh filename=meshes/wrist_flex_link_collision_2.stl; visual mesh filename=meshes/wrist_flex_link.dae
- link wrist_roll_link: geometry collision mesh filename=meshes/wrist_roll_link_collision_2.stl; visual mesh filename=meshes/wrist_roll_link.dae

File: resources/fetch/fetch_spherized.urdf (robot description, URDF)
Before this commit: robot fetch, 17 links, 16 joints
Links:
- link base_link: geometry collision sphere radius=0.066; collision sphere radius=0.066
- link bellows_link: geometry visual mesh filename=meshes/bellows_link.STL
- link elbow_flex_link: geometry collision sphere radius=0.03; collision sphere radius=0.03
- link forearm_roll_link: geometry collision sphere radius=0.03; collision sphere radius=0.03
- link gripper_link: geometry collision sphere radius=0.05; collision sphere radius=0.05
- link head_pan_link: geometry collision sphere radius=0.03; collision sphere radius=0.03
- link head_tilt_link: geometry visual mesh filename=meshes/head_tilt_link.dae
- link l_gripper_finger_link: geometry collision sphere radius=0.012; collision sphere radius=0.012
- link r_gripper_finger_link: geometry collision sphere radius=0.012; collision sphere radius=0.012
- link shoulder_lift_link: geometry collision sphere radius=0.04; collision sphere radius=0.04
- link shoulder_pan_link: geometry collision sphere radius=0.055; collision sphere radius=0.055
- link torso_fixed_link: geometry collision sphere radius=0.12; collision sphere radius=0.12
- link torso_lift_link: geometry collision sphere radius=0.15; collision sphere radius=0.15
- link upperarm_roll_link: geometry collision sphere radius=0.03; collision sphere radius=0.03
- link wrist_flex_link: geometry collision sphere radius=0.03; collision sphere radius=0.03
- link wrist_roll_link: geometry collision sphere radius=0.055; collision sphere radius=0.055
